File: AS3340-VCO.kicad_pcb (KiCad board)
At the start: 2 copper layers, 90.9 x 101.6 mm, 61 parts, among them J1 1V/OCT_INPUT, J10 SAWTOOTH_OUT, J11 TRIANGLE_OUT, J2 1V/OCT_OUT, J3 CV2_INPUT, J4 EXT_PWM_CTRL_INPUT, J5 POSITIVE_HARD_SYNC_INPUT, J6 NEGATIVE_HARD_SYNC_INPUT, J7 SOFT_SYNC_INPUT, J8 FM_INPUT, J9 SQUARE_OUT, SW1 SW_SPDT, U1 TL074, U2 AS3340

Commit message: Refactor
Parts:
- added BOTTOM_LEFT_MOUNT: MountingHole_3.2mm_M3_Oval, Seattle_Synths:MountingHole_3.2mm_M3_Oval, F.Cu at (115.9, 154.2)
- added BOTTOM_RIGHT_MOUNT: MountingHole_3.2mm_M3_Oval, Seattle_Synths:MountingHole_3.2mm_M3_Oval, F.Cu at (172.1, 154.2)
- added TOP_LEFT_MOUNT: MountingHole_3.2mm_M3_Oval, Seattle_Synths:MountingHole_3.2mm_M3_Oval, F.Cu at (116.0, 27.0)
- added TOP_RIGHT_MOUNT: MountingHole_3.2mm_M3_Oval, Seattle_Synths:MountingHole_3.2mm_M3_Oval, F.Cu at (172.1, 27.0)
- J5: value POSITIVE_HARD_SYNC_INPUT -> POS_HARD_SYNC_INPUT
- J6: value NEGATIVE_HARD_SYNC_INPUT -> NEG_HARD_SYNC_INPUT
- moved TP1 103.5 mm to (173.3, 36.8), turned to 270 degrees
- moved TP2 96.5 mm to (173.4, 42.7), turned to 270 degrees
- moved TP3 89.2 mm to (173.4, 49.0), turned to 90 degrees
- moved SW1 67.3 mm to (144.6, 116.4)
- moved C5 60.1 mm to (160.7, 29.6)
- moved U1 58.2 mm to (150.5, 59.8), turned to 90 degrees
- moved U2 53.3 mm to (122.3, 59.8), turned to 90 degrees
- moved R24 50.2 mm to (166.5, 149.2)
- moved R20 50.2 mm to (166.5, 128.6)
- moved R21 50.2 mm to (166.5, 133.8)
- moved R22 50.2 mm to (166.3, 138.9)
- moved R23 50.2 mm to (166.3, 144.0)
- moved D1 48.9 mm to (167.1, 101.3)
- moved C6 48.9 mm to (168.6, 88.1)
- moved C7 48.9 mm to (168.3, 94.8)
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Routing:
- net GND: track 394.2 -> 0.00 mm
- net +12V: track 261.1 -> 0.00 mm
- net -12V: track 206.1 -> 0.00 mm
- net Net-(R13-Pad1): track 164.5 -> 0.00 mm
- net /FREQ_CTRL: track 156.2 -> 0.00 mm
- net Net-(R17-Pad2): track 100.6 -> 0.00 mm, vias 1 -> 0
- net Net-(J1-PadT): track 97.7 -> 0.00 mm
- net Net-(R5-Pad1): track 88.8 -> 0.00 mm
- net /SAWTOOTH_OUT: track 86.8 -> 0.00 mm
- net Net-(C2-Pad2): track 84.0 -> 0.00 mm
- net Net-(C3-Pad2): track 82.9 -> 0.00 mm
- net Net-(R18-Pad2): track 81.5 -> 0.00 mm
- net /LINEAR_FM: track 74.9 -> 0.00 mm
- net Net-(R23-Pad2): track 74.0 -> 0.00 mm
- net /SOFT_SYNC: track 73.7 -> 0.00 mm, vias 1 -> 0
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Other:
- board size 90.9 x 101.6 mm -> 71 x 133.2 mm

Commit message: Refactor
Parts:
- added C10: 10uF, Seattle_Synths:CP_Radial_D5.0mm_P2.50mm, F.Cu at (138.7, 126.0)
- added C11: .1uF, Seattle_Synths:CP_Radial_D5.0mm_P2.50mm, F.Cu at (146.0, 126.3)
- added C8: 10uF, Seattle_Synths:CP_Radial_D5.0mm_P2.50mm, F.Cu at (138.6, 103.4)
- added C9: .1uF, Seattle_Synths:CP_Radial_D5.0mm_P2.50mm, F.Cu at (146.0, 103.2)
- added D4: LED, Seattle_Synths:LED_D5.0mm, F.Cu at (115.3, 35.2)
- added J12: EURO_PWR_2x5, Seattle_Synths:PinHeader_2x05_P2.54mm_Vertical, F.Cu at (173.8, 58.3)
- added R27: 330R, Seattle_Synths:R_Axial_DIN0207_L6.3mm_D2.5mm_P10.16mm_Horizontal, F.Cu at (165.4, 47.1)
- C1, C2, C3, C4, C5, C7: footprint SeattleSynths:C_Disc_D7.5mm_W2.5mm_P5.00mm -> Seattle_Synths:C_Disc_D7.5mm_W2.5mm_P5.00mm
- C6: value 500pF -> 500pF (Styrene); footprint SeattleSynths:C_Disc_D7.5mm_W2.5mm_P5.00mm -> Seattle_Synths:C_Disc_D7.5mm_W2.5mm_P5.00mm
- D1, D2: footprint Diode_THT:D_DO-35_SOD27_P7.62mm_Horizontal -> Seattle_Synths:D_DO-35_SOD27_P7.62mm_Horizontal
- D3: value D_Zener -> Zener 10V; footprint Diode_THT:D_DO-35_SOD27_P7.62mm_Horizontal -> Seattle_Synths:D_DO-35_SOD27_P7.62mm_Horizontal
- J1, J10, J11, J2, J3, J4, J5, J6, J7, J8, J9: footprint SeattleSynths:Jack_3.5mm_QingPu_WQP-PJ398SM_Vertical_CircularHoles -> Seattle_Synths:Jack_3.5mm_QingPu_WQP-PJ398SM_Vertical_CircularHoles
- R1, R10, R11, R12, R13, R14, R15, R16, R17, R18, R19, R2, R20, R21, R22, R23, R24, R25, R26, R3, R4, R5, R6, R7, R8, R9: footprint SeattleSynths:R_Axial_DIN0207_L6.3mm_D2.5mm_P10.16mm_Horizontal -> Seattle_Synths:R_Axial_DIN0207_L6.3mm_D2.5mm_P10.16mm_Horizontal
- RV1, RV2, RV3, RV5, RV8: footprint SeattleSynths:Potentiometer_Alpha_RD901F-40-00D_Single_Vertical -> Seattle_Synths:Potentiometer_Alpha_RD901F-40-00D_Single_Vertical
- RV4, RV6, RV7: footprint Potentiometer_THT:Potentiometer_Runtron_RM-065_Vertical -> Seattle_Synths:Potentiometer_Runtron_RM-065_Vertical
- U2: footprint Package_DIP:DIP-16_W7.62mm -> Seattle_Synths:DIP-16_W7.62mm
- moved RV7 7.41 mm to (164.7, 66.8)
- moved RV4 3.21 mm to (168.5, 77.3)

Commit message: Refactor
Parts:
- C11, C9: value .1uF -> 100nF; footprint Seattle_Synths:CP_Radial_D5.0mm_P2.50mm -> Seattle_Synths:C_Disc_D7.5mm_W2.5mm_P5.00mm
- D4, J10, J11, J2, J3, J9, RV1, RV2, RV3, RV5, RV8: moved to B.Cu
- J1: value 1V/OCT_INPUT -> 1V/OCT_IN; moved to B.Cu
- J4: value EXT_PWM_CTRL_INPUT -> EXT_PWM_CTRL_IN; moved to B.Cu
- J5: value POS_HARD_SYNC_INPUT -> POS_HARD_SYNC_IN; moved to B.Cu
- J6: value NEG_HARD_SYNC_INPUT -> NEG_HARD_SYNC_IN; moved to B.Cu
- J7: value SOFT_SYNC_INPUT -> SOFT_SYNC_IN; moved to B.Cu
- J8: value FM_INPUT -> FM_IN; moved to B.Cu
- SW1: footprint Button_Switch_THT:SW_Slide_1P2T_CK_OS102011MS2Q -> Seattle_Synths:SW_Toggle_Blue_wSlots; moved to B.Cu
- U1: footprint Package_DIP:DIP-14_W7.62mm -> Seattle_Synths:DIP-14_W7.62mm_Socket
- U2: footprint Seattle_Synths:DIP-16_W7.62mm -> Seattle_Synths:DIP-16_W7.62mm_Socket
- moved R25 25.3 mm to (166.8, 143.7)
- moved R26 25.3 mm to (166.8, 148.8)
- moved RV7 22.3 mm to (142.4, 67.1)
- moved R27 20.4 mm to (145.0, 46.6)
- moved R23 10.5 mm to (166.7, 133.5)
- moved R24 10.5 mm to (166.9, 138.7)
- moved R22 10.5 mm to (166.7, 128.4)
- moved R20 10.5 mm to (166.9, 118.1)
- moved R21 10.5 mm to (166.9, 123.3)
- moved RV1 6.78 mm to (159.7, 47.5)
- moved RV8 6.53 mm to (159.6, 75.8)
- moved RV3 5.61 mm to (147.6, 94.6)
- moved RV5 2.70 mm to (135.0, 47.4)
- moved RV2 2.59 mm to (135.0, 75.9)
- moved U2 1.98 mm to (124.2, 60.4)
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
Commit message: Refactor
Parts:
- moved C10 0.45 mm to (139.3, 127.8)
- moved C8 0.21 mm to (139.3, 102.0)
Connections:
- C10 pad 1: GND -> +12V
- C10 pad 2: +12V -> GND
- C8 pad 1: -12V -> GND
- C8 pad 2: GND -> -12V
Other:
- board text added: "Seattle Synths SS-VCO-1 (C) 2020 Nate Houk Rev. 1"
