File: AS3340-VCO.kicad_pcb (KiCad board)
At the start: 2 copper layers, 71 x 133.2 mm, 72 parts, among them J1 1V/OCT_IN, J10 SAWTOOTH_OUT, J11 TRIANGLE_OUT, J12 -----, J2 1V/OCT_OUT, J3 CV2_INPUT, J4 EXT_PWM_CTRL_IN, J5 POS_HARD_SYNC_IN, J6 NEG_HARD_SYNC_IN, J7 SOFT_SYNC_IN, J8 FM_IN, J9 SQUARE_OUT, SW1 SW_SPDT, U1 TL074, U2 AS3340

Commit message: Refactor
Parts:
- moved R16 5.12 mm to (113.8, 128.9)
- moved C10 5.12 mm to (141.4, 123.1)
- moved C11 5.12 mm to (148.0, 122.8)
- moved C9 5.12 mm to (147.8, 97.1)
- moved D1 5.12 mm to (169.6, 96.6)
- moved J1 5.12 mm to (132.9, 75.0)
- moved J3 5.12 mm to (132.9, 90.1)
- moved J4 5.12 mm to (132.9, 105.1)
- moved R22 5.12 mm to (168.8, 123.7)
- moved R7 5.12 mm to (113.8, 83.0)
- moved RV7 5.12 mm to (144.4, 62.4)
- moved TP1 5.12 mm to (175.4, 32.1)
- moved U2 5.12 mm to (126.3, 55.7)
- moved C1 5.12 mm to (125.1, 24.9)
- moved C2 5.12 mm to (134.6, 24.9)
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
Commit message: Rev. 1
Parts:
- J12: value ----- -> EURO_PWR_2x5
- RV4, RV6, RV7: footprint Seattle_Synths:Potentiometer_Runtron_RM-065_Vertical -> Seattle_Synths:TRIM_3266W-1-102LF
- moved RV7 5.55 mm to (146.5, 67.5)
- moved RV6 5.40 mm to (117.7, 53.1)
- moved RV4 3.18 mm to (173.9, 74.2)
Routing:
- net +12V: track 238.5 -> 264.9 mm
- net Net-(C2-Pad2): track 133.8 -> 159.3 mm
- net Net-(C3-Pad2): track 126.2 -> 143.1 mm
- net GND: track 446.0 -> 430.7 mm
- net /SOFT_SYNC: track 59.9 -> 68.7 mm, vias 1 -> 0
- net Net-(R13-Pad1): track 124.8 -> 116.0 mm, vias 0 -> 1
- net Net-(R5-Pad1): track 76.8 -> 85.6 mm
- net Net-(R1-Pad1): track 86.7 -> 79.8 mm, vias 0 -> 1
- net Net-(RV5-Pad2): track 87.3 -> 80.5 mm, vias 1 -> 0
- net Net-(R12-Pad2): track 68.1 -> 62.4 mm
- net Net-(RV7-Pad1): track 7.91 -> 12.9 mm
- net Net-(C3-Pad1): track 130.7 -> 125.9 mm
- net /SQUARE: track 83.7 -> 79.6 mm, vias 0 -> 1
- net Net-(J4-PadT): track 85.7 -> 89.5 mm, vias 1 -> 0
- net Net-(C6-Pad2): track 58.3 -> 54.6 mm
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
Commit message: Refactor
Parts:
- J12: footprint Seattle_Synths:PinHeader_2x05_P2.54mm_Vertical -> Seattle_Synths:3M_2510-6002UB
- TP1, TP2, TP3: footprint SeattleSynths:TestPoint_Pad_4.0x4.0mm -> Seattle_Synths:TestPoint_Pad_4.0x4.0mm
- moved J9 30.3 mm to (131.0, 137.1)
- moved J10 30.1 mm to (131.0, 122.1)
- moved J5 28.1 mm to (161.0, 136.8)
- moved J7 28.1 mm to (161.0, 121.8)
- moved R27 10.3 mm to (147.0, 31.6), turned to 270 degrees
- moved R19 10.0 mm to (123.7, 144.2), turned to 180 degrees
- moved J12 7.20 mm to (175.1, 60.1), turned to 270 degrees
- moved J6 4.30 mm to (146.0, 133.9)
- moved RV4 2.69 mm to (174.5, 76.8)
- moved J3 2.64 mm to (130.8, 91.7)
- moved J4 2.64 mm to (130.8, 106.7)
- moved J1 2.36 mm to (130.8, 76.1)
- moved RV3 2.01 mm to (148.5, 88.2)
- moved SW1 1.26 mm to (146.0, 110.1)
- moved U2 0.90 mm to (125.5, 55.2)
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Routing:
- net GND: track 430.7 -> 0.00 mm
- net +12V: track 264.9 -> 0.00 mm
- net -12V: track 203.9 -> 0.00 mm
- net Net-(C2-Pad2): track 159.3 -> 0.00 mm
- net Net-(C5-Pad2): track 150.8 -> 0.00 mm
- net Net-(C3-Pad2): track 143.1 -> 0.00 mm
- net Net-(C2-Pad1): track 140.7 -> 0.00 mm
- net Net-(C4-Pad2): track 135.3 -> 0.00 mm
- net Net-(C3-Pad1): track 125.9 -> 0.00 mm
- net Net-(R13-Pad1): track 116.0 -> 0.00 mm, vias 1 -> 0
- net /FREQ_CTRL: track 111.7 -> 0.00 mm
- net Net-(R23-Pad2): track 99.5 -> 0.00 mm
- net Net-(R26-Pad2): track 98.0 -> 0.00 mm
- net Net-(R18-Pad2): track 97.4 -> 0.00 mm
- net Net-(R22-Pad2): track 96.2 -> 0.00 mm
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Other:
- board text added: "Seattle Synths SS-VCO-1 Rev. 2 [2020-11-15]"
- board text removed: "Seattle Synths SS-VCO-1 Rev. 1 [2020-11-08]"

Commit message: Revv. 2
Parts:
- removed TP1: +12V, Seattle_Synths:TestPoint_Pad_4.0x4.0mm
- removed TP2: GND, Seattle_Synths:TestPoint_Pad_4.0x4.0mm
- removed TP3: -12V, Seattle_Synths:TestPoint_Pad_4.0x4.0mm
- C1, C11, C2, C3, C4, C5, C7, C9: footprint Seattle_Synths:C_Disc_D7.5mm_W2.5mm_P5.00mm -> Seattle_Synths:C_0603_1608Metric
- D4: footprint Seattle_Synths:LED_D5.0mm -> Seattle_Synths:D_0603_1608Metric
- R1, R10, R11, R12, R13, R14, R15, R16, R17, R18, R19, R2, R20, R21, R22, R23, R24, R25, R26, R27, R3, R4, R5, R6, R7, R8, R9: footprint Seattle_Synths:R_Axial_DIN0207_L6.3mm_D2.5mm_P10.16mm_Horizontal -> Seattle_Synths:R_0603_1608Metric
- RV1: value 100K -> 100K (Fine)
- RV2: value 100K -> 100K (CV2)
- RV3: value 100K -> 100K (PWM)
- RV5: value 100K -> 100K (Pitch)
- RV8: value 100K -> 100K (FM)
- moved R1 106.7 mm to (126.0, 143.3)
- moved C3 98.9 mm to (161.0, 122.4)
- moved R16 97.7 mm to (145.8, 36.6)
- moved R14 93.4 mm to (154.9, 34.8), turned to 180 degrees
- moved R15 84.8 mm to (140.2, 43.2), turned to 180 degrees
- moved U2 84.4 mm to (121.7, 139.4), turned to 180 degrees
- moved R17 75.9 mm to (170.2, 83.3)
- moved C11 73.3 mm to (149.6, 49.5)
- moved U1 71.4 mm to (170.9, 124.2), turned to 0 degrees
- moved RV6 68.9 mm to (176.8, 88.5), turned to 90 degrees
- moved R8 68.2 mm to (154.4, 142.7), turned to 180 degrees
- moved R10 65.8 mm to (176.3, 118.9)
- moved C10 62.7 mm to (173.2, 69.1)
- moved R2 58.2 mm to (120.4, 100.1), turned to 90 degrees
- moved R12 56.5 mm to (166.6, 88.6)
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Routing:
- net GND: track 0.00 -> 388.5 mm
- net +12V: track 0.00 -> 259.4 mm
- net /FREQ_CTRL: track 0.00 -> 212.9 mm
- net -12V: track 0.00 -> 185.5 mm, vias 0 -> 1
- net /LINEAR_FM: track 0.00 -> 130.1 mm
- net Net-(R13-Pad1): track 0.00 -> 120.6 mm, vias 0 -> 1
- net /PWM: track 0.00 -> 94.3 mm, vias 0 -> 1
- net Net-(RV7-Pad1): track 0.00 -> 92.5 mm
- net Net-(R12-Pad1): track 0.00 -> 90.3 mm, vias 0 -> 1
- net Net-(R1-Pad1): track 0.00 -> 90.1 mm
- net Net-(J4-PadT): track 0.00 -> 83.2 mm
- net Net-(J1-PadT): track 0.00 -> 75.6 mm
- net Net-(D3-Pad1): track 0.00 -> 72.1 mm, vias 0 -> 1
- net Net-(C6-Pad2): track 0.00 -> 71.7 mm
- net /HARD_SYNC: track 0.00 -> 71.4 mm
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Other:
- board size 71 x 133.2 mm -> 71 x 128.9 mm
