File: AS3340-VCO.sch (KiCad schematic (older format))
At the start: 61 parts, among them J1 1V/OCT_INPUT, J10 SAWTOOTH_OUT, J11 TRIANGLE_OUT, J2 1V/OCT_OUT, J3 CV2_INPUT, J4 EXT_PWM_CTRL_INPUT, J5 POSITIVE_HARD_SYNC_INPUT, J6 NEGATIVE_HARD_SYNC_INPUT, J7 SOFT_SYNC_INPUT, J8 FM_INPUT, J9 SQUARE_OUT, SW1 SW_SPDT, U1 TL074, U2 AS3340

Commit message: Refactor
Parts:
- added C10, C8: 10uF, Seattle_Synths:CP_Radial_D5.0mm_P2.50mm, symbol Device:C
- added C11, C9: .1uF, Seattle_Synths:CP_Radial_D5.0mm_P2.50mm, symbol Device:C
- added J12: EURO_PWR_2x5, Seattle_Synths:PinHeader_2x05_P2.54mm_Vertical, symbol Seattle_Synths:EURO_PWR_2x5
- D1, D2, D3: footprint Diode_THT:D_DO-35_SOD27_P7.62mm_Horizontal -> Seattle_Synths:D_DO-35_SOD27_P7.62mm_Horizontal
Connections:
- net +12V: now also C10.2, C11.2, J12.1 (+12V), J12.2 (+12V)
- net -12V: now also C8.1, C9.1, J12.10 (-12V), J12.9 (-12V)
- net GND: now also C10.1, C11.1, C8.2, C9.2, J12.3 (GND), J12.4 (GND), J12.5 (GND), J12.6 (GND), J12.7 (GND), J12.8 (GND)
Other:
- moved on the sheet: C1, J1, J2, J3, J4, R1, R10, R11, R2, R3, R4, R5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

Commit message: Refactor
Parts:
- added D4: LED, symbol Device:LED
- added R27: 330R, symbol Device:R
Connections:
- net +12V: now also R27.2
- net GND: now also D4.1 (K)
- new net: D4.2 (A), R27.1
Other:
- moved on the sheet: C10, C11, C8, C9, J12, TP1, TP2, TP3, U1E

Commit message: Refactor
Changed lines of the file:
@@
 Wire Wire Line
 	4500 3250 4500 3200
-Wire Wire Line
-	7200 3050 7200 2750
 $Comp
 L power:+12V #PWR026
@@
 	0    1    1    0
 $EndComp
-$Comp
-L power:PWR_FLAG #FLG02
-U 1 1 5F954D5F
-P 7500 2750
-F 0 "#FLG02" H 7500 2825 50  0001 C CNN
-F 1 "PWR_FLAG" V 7500 2878 50  0000 L CNN
-F 2 "" H 7500 2750 50  0001 C CNN
-F 3 "~" H 7500 2750 50  0001 C CNN
-	1    7500 2750
-	0    1    1    0
-$EndComp
-Wire Wire Line
-	7500 2750 7200 2750
-Connection ~ 7200 2750
-Wire Wire Line
-	7200 2750 7200 2700
 NoConn ~ 9400 5200
 NoConn ~ 9400 4550
@@
 	-1   0    0    1
 $EndComp
+Wire Wire Line
+	7200 2700 7200 3050
 $EndSCHEMATC

Commit message: Refactor
Parts:
- C1, C2, C3, C4, C5, C6, C7: footprint SeattleSynths:C_Disc_D7.5mm_W2.5mm_P5.00mm -> Seattle_Synths:C_Disc_D7.5mm_W2.5mm_P5.00mm
- D4: footprint (none) -> Seattle_Synths:LED_D5.0mm
- J1, J10, J11, J2, J3, J4, J7, J8, J9: footprint SeattleSynths:Jack_3.5mm_QingPu_WQP-PJ398SM_Vertical_CircularHoles -> Seattle_Synths:Jack_3.5mm_QingPu_WQP-PJ398SM_Vertical_CircularHoles
- J5: value POSITIVE_HARD_SYNC_INPUT -> POS_HARD_SYNC_INPUT; footprint SeattleSynths:Jack_3.5mm_QingPu_WQP-PJ398SM_Vertical_CircularHoles -> Seattle_Synths:Jack_3.5mm_QingPu_WQP-PJ398SM_Vertical_CircularHoles
- J6: value NEGATIVE_HARD_SYNC_INPUT -> NEG_HARD_SYNC_INPUT; footprint SeattleSynths:Jack_3.5mm_QingPu_WQP-PJ398SM_Vertical_CircularHoles -> Seattle_Synths:Jack_3.5mm_QingPu_WQP-PJ398SM_Vertical_CircularHoles
- R1, R10, R11, R12, R13, R14, R15, R16, R17, R18, R19, R2, R20, R21, R22, R23, R24, R25, R26, R3, R4, R5, R6, R7, R8, R9: footprint SeattleSynths:R_Axial_DIN0207_L6.3mm_D2.5mm_P10.16mm_Horizontal -> Seattle_Synths:R_Axial_DIN0207_L6.3mm_D2.5mm_P10.16mm_Horizontal
- R27: footprint (none) -> Seattle_Synths:R_Axial_DIN0207_L6.3mm_D2.5mm_P10.16mm_Horizontal
- RV1, RV2, RV3, RV5, RV8: footprint SeattleSynths:Potentiometer_Alpha_RD901F-40-00D_Single_Vertical -> Seattle_Synths:Potentiometer_Alpha_RD901F-40-00D_Single_Vertical
- RV4, RV6, RV7: footprint Potentiometer_THT:Potentiometer_Runtron_RM-065_Vertical -> Seattle_Synths:Potentiometer_Runtron_RM-065_Vertical
- U2: footprint Package_DIP:DIP-16_W7.62mm -> Seattle_Synths:DIP-16_W7.62mm

Commit message: Refactor
Parts:
- C11, C9: value .1uF -> 100nF; footprint Seattle_Synths:CP_Radial_D5.0mm_P2.50mm -> Seattle_Synths:C_Disc_D7.5mm_W2.5mm_P5.00mm
- J1: value 1V/OCT_INPUT -> 1V/OCT_IN
- J4: value EXT_PWM_CTRL_INPUT -> EXT_PWM_CTRL_IN
- J5: value POS_HARD_SYNC_INPUT -> POS_HARD_SYNC_IN
- J6: value NEG_HARD_SYNC_INPUT -> NEG_HARD_SYNC_IN
- J7: value SOFT_SYNC_INPUT -> SOFT_SYNC_IN
- J8: value FM_INPUT -> FM_IN
- SW1: footprint Button_Switch_THT:SW_Slide_1P2T_CK_OS102011MS2Q -> Seattle_Synths:SW_Toggle_Blue_wSlots
- U1: footprint Package_DIP:DIP-14_W7.62mm -> Seattle_Synths:DIP-14_W7.62mm_Socket
- U2: footprint Seattle_Synths:DIP-16_W7.62mm -> Seattle_Synths:DIP-16_W7.62mm_Socket
Changed lines of the file:
@@
 F 0 "U1" H 9450 2417 50  0000 C CNN
 F 1 "TL074" H 9450 2326 50  0000 C CNN
-F 2 "Package_DIP:DIP-14_W7.62mm" H 9400 2150 50  0001 C CNN
+F 2 "Seattle_Synths:DIP-14_W7.62mm_Socket" H 9400 2150 50  0001 C CNN
 F 3 "http://www.ti.com/lit/ds/symlink/tl071.pdf" H 9500 2250 50  0001 C CNN
 	1    9450 2050
@@
 F 0 "U1" H 9450 1467 50  0000 C CNN
 F 1 "TL074" H 9450 1376 50  0000 C CNN
-F 2 "Package_DIP:DIP-14_W7.62mm" H 9400 1200 50  0001 C CNN
+F 2 "Seattle_Synths:DIP-14_W7.62mm_Socket" H 9400 1200 50  0001 C CNN
 F 3 "http://www.ti.com/lit/ds/symlink/tl071.pdf" H 9500 1300 50  0001 C CNN
 	2    9450 1100
@@
 F 0 "U1" H 5400 7117 50  0000 C CNN
 F 1 "TL074" H 5400 7026 50  0000 C CNN
-F 2 "Package_DIP:DIP-14_W7.62mm" H 5350 6850 50  0001 C CNN
+F 2 "Seattle_Synths:DIP-14_W7.62mm_Socket" H 5350 6850 50  0001 C CNN
 F 3 "http://www.ti.com/lit/ds/symlink/tl071.pdf" H 5450 6950 50  0001 C CNN
 	4    5400 6750
@@
 P 3950 7050
 F 0 "J4" H 3770 6983 50  0000 R CNN
-F 1 "EXT_PWM_CTRL_INPUT" H 3770 7074 50  0000 R CNN
+F 1 "EXT_PWM_CTRL_IN" H 3770 7074 50  0000 R CNN
 F 2 "Seattle_Synths:Jack_3.5mm_QingPu_WQP-PJ398SM_Vertical_CircularHoles" H 3950 7050 50  0001 C CNN
 F 3 "~" H 3950 7050 50  0001 C CNN
@@
 F 0 "U1" H 9450 3367 50  0000 C CNN
 F 1 "TL074" H 9450 3276 50  0000 C CNN
-F 2 "Package_DIP:DIP-14_W7.62mm" H 9400 3100 50  0001 C CNN
+F 2 "Seattle_Synths:DIP-14_W7.62mm_Socket" H 9400 3100 50  0001 C CNN
 F 3 "http://www.ti.com/lit/ds/symlink/tl071.pdf" H 9500 3200 50  0001 C CNN
 	3    9450 3000
@@
 P 6150 1050
 F 0 "J8" H 5970 983 50  0000 R CNN
-F 1 "FM_INPUT" H 5970 1074 50  0000 R CNN
+F 1 "FM_IN" H 5970 1074 50  0000 R CNN
 F 2 "Seattle_Synths:Jack_3.5mm_QingPu_WQP-PJ398SM_Vertical_CircularHoles" H 6150 1050 50  0001 C CNN
 F 3 "~" H 6150 1050 50  0001 C CNN
@@
 P 1800 1450
 F 0 "J1" H 1620 1383 50  0000 R CNN
-F 1 "1V/OCT_INPUT" H 1620 1474 50  0000 R CNN
+F 1 "1V/OCT_IN" H 1620 1474 50  0000 R CNN
 F 2 "Seattle_Synths:Jack_3.5mm_QingPu_WQP-PJ398SM_Vertical_CircularHoles" H 1800 1450 50  0001 C CNN
 F 3 "~" H 1800 1450 50  0001 C CNN
@@
 F 0 "SW1" H 1450 3535 50  0000 C CNN
 F 1 "SW_SPDT" H 1450 3444 50  0000 C CNN
-F 2 "Button_Switch_THT:SW_Slide_1P2T_CK_OS102011MS2Q" H 1450 3250 50  0001 C CNN
+F 2 "Seattle_Synths:SW_Toggle_Blue_wSlots" H 1450 3250 50  0001 C CNN
 F 3 "~" H 1450 3250 50  0001 C CNN
 	1    1450 3250
@@
 P 5800 5900
 F 0 "J7" H 5832 6225 50  0000 C CNN
-F 1 "SOFT_SYNC_INPUT" H 5832 6134 50  0000 C CNN
+F 1 "SOFT_SYNC_IN" H 5832 6134 50  0000 C CNN
 F 2 "Seattle_Synths:Jack_3.5mm_QingPu_WQP-PJ398SM_Vertical_CircularHoles" H 5800 5900 50  0001 C CNN
 F 3 "~" H 5800 5900 50  0001 C CNN
@@
 F 0 "U2" H 7200 4631 50  0000 C CNN
 F 1 "AS3340" H 7200 4540 50  0000 C CNN
-F 2 "Seattle_Synths:DIP-16_W7.62mm" H 7700 3450 50  0001 C CNN
+F 2 "Seattle_Synths:DIP-16_W7.62mm_Socket" H 7700 3450 50  0001 C CNN
 F 3 "http://www.alfarzpp.lv/eng/sc/AS3340.pdf" H 7800 3300 50  0001 C CNN
 	1    7200 3750
@@
 F 0 "U1" H 1708 7046 50  0000 L CNN
 F 1 "TL074" H 1708 6955 50  0000 L CNN
-F 2 "Package_DIP:DIP-14_W7.62mm" H 1700 7100 50  0001 C CNN
+F 2 "Seattle_Synths:DIP-14_W7.62mm_Socket" H 1700 7100 50  0001 C CNN
 F 3 "http://www.ti.com/lit/ds/symlink/tl071.pdf" H 1800 7200 50  0001 C CNN
 	5    1750 7000
@@
 P 3150 5500
 F 0 "J6" H 3182 5825 50  0000 C CNN
-F 1 "NEG_HARD_SYNC_INPUT" H 3182 5734 50  0000 C CNN
+F 1 "NEG_HARD_SYNC_IN" H 3182 5734 50  0000 C CNN
 F 2 "Seattle_Synths:Jack_3.5mm_QingPu_WQP-PJ398SM_Vertical_CircularHoles" H 3150 5500 50  0001 C CNN
 F 3 "~" H 3150 5500 50  0001 C CNN
@@
 P 3150 4900
 F 0 "J5" H 3182 5225 50  0000 C CNN
-F 1 "POS_HARD_SYNC_INPUT" H 3182 5134 50  0000 C CNN
+F 1 "POS_HARD_SYNC_IN" H 3182 5134 50  0000 C CNN
 F 2 "Seattle_Synths:Jack_3.5mm_QingPu_WQP-PJ398SM_Vertical_CircularHoles" H 3150 4900 50  0001 C CNN
 F 3 "~" H 3150 4900 50  0001 C CNN
@@
 P 1300 6900
 F 0 "C9" V 1048 6900 50  0000 C CNN
-F 1 ".1uF" V 1139 6900 50  0000 C CNN
-F 2 "Seattle_Synths:CP_Radial_D5.0mm_P2.50mm" H 1338 6750 50  0001 C CNN
+F 1 "100nF" V 1139 6900 50  0000 C CNN
+F 2 "Seattle_Synths:C_Disc_D7.5mm_W2.5mm_P5.00mm" H 1338 6750 50  0001 C CNN
 F 3 "~" H 1300 6900 50  0001 C CNN
 	1    1300 6900
@@
 P 2200 6900
 F 0 "C11" V 1948 6900 50  0000 C CNN
-F 1 ".1uF" V 2039 6900 50  0000 C CNN
-F 2 "Seattle_Synths:CP_Radial_D5.0mm_P2.50mm" H 2238 6750 50  0001 C CNN
+F 1 "100nF" V 2039 6900 50  0000 C CNN
+F 2 "Seattle_Synths:C_Disc_D7.5mm_W2.5mm_P5.00mm" H 2238 6750 50  0001 C CNN
 F 3 "~" H 2200 6900 50  0001 C CNN
 	1    2200 6900

Commit message: Refactor
Parts:
- removed C10, C8: 10uF, Seattle_Synths:CP_Radial_D5.0mm_P2.50mm, symbol Device:C
- added C10, C8: 10uF, Seattle_Synths:CP_Radial_D5.0mm_P2.50mm, symbol Device:C_Polarized
Connections:
- net +12V: now also C10.1
- net -12V: now also C8.2
- net GND: now also C10.2, C8.1
Changed lines of the file:
@@
-$EndComp
-$Comp
-L Device:C C8
-U 1 1 5FADF82D
-P 1300 6450
-F 0 "C8" V 1048 6450 50  0000 C CNN
-F 1 "10uF" V 1139 6450 50  0000 C CNN
-F 2 "Seattle_Synths:CP_Radial_D5.0mm_P2.50mm" H 1338 6300 50  0001 C CNN
-F 3 "~" H 1300 6450 50  0001 C CNN
-	1    1300 6450
-	0    1    1    0
 $EndComp
 $Comp
@@
 Wire Wire Line
 	1450 6450 1450 6000
-$Comp
-L Device:C C10
-U 1 1 5FB0085B
-P 2200 6450
-F 0 "C10" V 1948 6450 50  0000 C CNN
-F 1 "10uF" V 2039 6450 50  0000 C CNN
-F 2 "Seattle_Synths:CP_Radial_D5.0mm_P2.50mm" H 2238 6300 50  0001 C CNN
-F 3 "~" H 2200 6450 50  0001 C CNN
-	1    2200 6450
-	0    1    1    0
-$EndComp
 $Comp
 L power:+12V #PWR0116
@@
 Wire Wire Line
 	7200 2700 7200 3050
+$Comp
+L Device:C_Polarized C10
+U 1 1 5FB5200C
+P 2200 6450
+F 0 "C10" V 2455 6450 50  0000 C CNN
+F 1 "10uF" V 2364 6450 50  0000 C CNN
+F 2 "Seattle_Synths:CP_Radial_D5.0mm_P2.50mm" H 2238 6300 50  0001 C CNN
+F 3 "~" H 2200 6450 50  0001 C CNN
+	1    2200 6450
+	0    -1   -1   0
+$EndComp
+$Comp
+L Device:C_Polarized C8
+U 1 1 5FB5D9FF
+P 1300 6450
+F 0 "C8" V 1555 6450 50  0000 C CNN
+F 1 "10uF" V 1464 6450 50  0000 C CNN
+F 2 "Seattle_Synths:CP_Radial_D5.0mm_P2.50mm" H 1338 6300 50  0001 C CNN
+F 3 "~" H 1300 6450 50  0001 C CNN
+	1    1300 6450
+	0    -1   -1   0
+$EndComp
 $EndSCHEMATC

Commit message: Rev. 1
Parts:
- J12: footprint Seattle_Synths:PinHeader_2x05_P2.54mm_Vertical -> Seattle_Synths:61201021621
- RV4, RV6, RV7: footprint Seattle_Synths:Potentiometer_Runtron_RM-065_Vertical -> Seattle_Synths:TRIM_3266W-1-102LF
- TP1, TP2, TP3: footprint SeattleSynths:TestPoint_Pad_4.0x4.0mm -> Seattle_Synths:TestPoint_Pad_4.0x4.0mm
Changed lines of the file:
@@
 F 0 "RV4" V 1535 900 50  0000 C CNN
 F 1 "100K" V 1444 900 50  0000 C CNN
-F 2 "Seattle_Synths:Potentiometer_Runtron_RM-065_Vertical" H 1650 900 50  0001 C CNN
+F 2 "Seattle_Synths:TRIM_3266W-1-102LF" H 1650 900 50  0001 C CNN
 F 3 "~" H 1650 900 50  0001 C CNN
 	1    1650 900
@@
 F 0 "RV7" V 5193 3650 50  0000 C CNN
 F 1 "10K" V 5284 3650 50  0000 C CNN
-F 2 "Seattle_Synths:Potentiometer_Runtron_RM-065_Vertical" H 5400 3650 50  0001 C CNN
+F 2 "Seattle_Synths:TRIM_3266W-1-102LF" H 5400 3650 50  0001 C CNN
 F 3 "~" H 5400 3650 50  0001 C CNN
 	1    5400 3650
@@
 F 0 "RV6" V 4385 3050 50  0000 C CNN
 F 1 "10K" V 4294 3050 50  0000 C CNN
-F 2 "Seattle_Synths:Potentiometer_Runtron_RM-065_Vertical" H 4500 3050 50  0001 C CNN
+F 2 "Seattle_Synths:TRIM_3266W-1-102LF" H 4500 3050 50  0001 C CNN
 F 3 "~" H 4500 3050 50  0001 C CNN
 	1    4500 3050
@@
 F 0 "TP1" V 1900 6400 50  0000 R CNN
 F 1 "+12V" V 2000 6400 50  0000 R CNN
-F 2 "SeattleSynths:TestPoint_Pad_4.0x4.0mm" H 2250 6000 50  0001 C CNN
+F 2 "Seattle_Synths:TestPoint_Pad_4.0x4.0mm" H 2250 6000 50  0001 C CNN
 F 3 "~" H 2250 6000 50  0001 C CNN
 	1    2050 6000
@@
 F 0 "TP2" H 1692 6376 50  0000 R CNN
 F 1 "GND" H 1692 6467 50  0000 R CNN
-F 2 "SeattleSynths:TestPoint_Pad_4.0x4.0mm" H 1950 6350 50  0001 C CNN
+F 2 "Seattle_Synths:TestPoint_Pad_4.0x4.0mm" H 1950 6350 50  0001 C CNN
 F 3 "~" H 1950 6350 50  0001 C CNN
 	1    1750 6350
@@
 F 0 "TP3" V 1550 6350 50  0000 R CNN
 F 1 "-12V" V 1450 6400 50  0000 R CNN
-F 2 "SeattleSynths:TestPoint_Pad_4.0x4.0mm" H 1650 6000 50  0001 C CNN
+F 2 "Seattle_Synths:TestPoint_Pad_4.0x4.0mm" H 1650 6000 50  0001 C CNN
 F 3 "~" H 1650 6000 50  0001 C CNN
 	1    1450 6000
@@
 F 0 "J12" H 3150 4247 60  0000 C CNN
 F 1 "EURO_PWR_2x5" H 3150 4141 60  0000 C CNN
-F 2 "Seattle_Synths:PinHeader_2x05_P2.54mm_Vertical" H 3150 3800 60  0001 C CNN
+F 2 "Seattle_Synths:61201021621" H 3150 3800 60  0001 C CNN
 F 3 "" H 3150 3800 60  0000 C CNN
 	1    3150 3800

Commit message: Refactor
Parts:
- J12: footprint Seattle_Synths:61201021621 -> Seattle_Synths:3M_2510-6002UB
Changed lines of the file:
@@
 F 0 "J12" H 3150 4247 60  0000 C CNN
 F 1 "EURO_PWR_2x5" H 3150 4141 60  0000 C CNN
-F 2 "Seattle_Synths:61201021621" H 3150 3800 60  0001 C CNN
+F 2 "Seattle_Synths:3M_2510-6002UB" H 3150 3800 60  0001 C CNN
 F 3 "" H 3150 3800 60  0000 C CNN
 	1    3150 3800
