File: AS3340-VCO.sch (KiCad schematic (older format))
At the start: 68 parts, among them J1 1V/OCT_IN, J10 SAWTOOTH_OUT, J11 TRIANGLE_OUT, J12 EURO_PWR_2x5, J2 1V/OCT_OUT, J3 CV2_INPUT, J4 EXT_PWM_CTRL_IN, J5 POS_HARD_SYNC_IN, J6 NEG_HARD_SYNC_IN, J7 SOFT_SYNC_IN, J8 FM_IN, J9 SQUARE_OUT, SW1 SW_SPDT, U1 TL074, U2 AS3340

Commit message: Revv. 2
Parts:
- C1, C11, C2, C3, C4, C5, C7, C9: footprint Seattle_Synths:C_Disc_D7.5mm_W2.5mm_P5.00mm -> Seattle_Synths:C_0603_1608Metric
- D4: footprint Seattle_Synths:LED_D5.0mm -> Seattle_Synths:D_0603_1608Metric
- R1, R10, R11, R12, R13, R14, R15, R16, R17, R18, R19, R2, R20, R21, R22, R23, R24, R25, R26, R27, R3, R4, R5, R6, R7, R8, R9: footprint Seattle_Synths:R_Axial_DIN0207_L6.3mm_D2.5mm_P10.16mm_Horizontal -> Seattle_Synths:R_0603_1608Metric
- RV1: value 100K -> 100K (Fine)
- RV2: value 100K -> 100K (CV2)
- RV3: value 100K -> 100K (PWM)
- RV5: value 100K -> 100K (Pitch)
- RV8: value 100K -> 100K (FM)
Other:
- moved on the sheet: J8
